File: PCB/PCB-Ange.kicad_pcb (KiCad board)
At the start: 2 copper layers, 75 x 75 mm, 54 parts, among them J1 Alim, J2 Conn_02x05_Odd_Even, J3 Conn_02x02_Odd_Even, Q1 Q_PMOS_GSD, Q2 Q_PMOS_GSD, Q3 Q_PMOS_GSD, SW1 SW_Push, SW2 SW_Push, SW3 SW_DIP_x01, U1 STM32F103C6Tx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

Commit message: Update du 25/08/22 à 07:56
Parts:
- moved J3 2.14 mm to (95.6, 126.6)
Routing:
- net JTMS-SWDIO: track 19.9 -> 24.1 mm
- net JTCK-SWCLK: track 17.6 -> 19.8 mm
- net GND: track 335.3 -> 334.7 mm
Other:
- outline, holes or cut-outs redrawn
- net class Default removed
